File: hardware/Electronic Speed Controller/ESC_KiCAD/pwr_usb_can.kicad_sch (KiCad schematic)
At the start: 40 parts, among them J4 XT60PW-M, J5 USB TYPE-A, U5 LM7805MPX/NOPB, U6 TPS54302DDCR, U7 LM66200DRLR, U8 TLV75533PDBVR

Commit message: finish ESC software state machine, refactor FCC sensor fusion and OTA packet reception. Create a common folder for shared code. i should commit more often lmao
Other:
- note added: "NOTES: DESIGNED FOR 4S, 6S BATTERIES 12.8 - 28V INPUT TOLERANT 3A CONTINUOUS"
- note removed: "NOTES: DESIGNED FOR 4S, 6S BATTERIES 12.8 - 28V INPUT TOLERANT MAX OUTPUT +10.94V, 2.05A CONTINUOUS"
Changed lines of the file:
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@@
 		)
 	)
-	(text "NOTES:\nDESIGNED FOR 4S, 6S BATTERIES\n12.8 - 28V INPUT TOLERANT\nMAX OUTPUT +10.94V, 2.05A CONTINUOUS"
+	(text "NOTES:\nDESIGNED FOR 4S, 6S BATTERIES\n12.8 - 28V INPUT TOLERANT\n3A CONTINUOUS"
 		(exclude_from_sim no)
 		(at 26.924 63.5 0)
